File: board/a2bikelight/a2bikelight.kicad_pcb (KiCad board)
At the start: 4 copper layers, 50 x 50 mm, 28 parts, among them J1 Barrel_Jack_Switch, J2 Conn_01x02_Male, J3 Conn_01x04_Male, J4 Conn_01x06_Male, J5 Conn_01x05_Male, SW1 SW_Push, SW2 SW_Push, U1 STM8L151K4U, U2 AMS1117-3.3, U3 MXC6655XA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

Commit message: layout
Parts:
- removed TP2: TestPoint, TestPoint:TestPoint_THTPad_2.0x2.0mm_Drill1.0mm
- added J6: Conn_01x08_Male, Connector_PinHeader_2.54mm:PinHeader_1x08_P2.54mm_Vertical, F.Cu at (146.7, 110.1)
- moved TP1 44.0 mm to (137.1, 105.4)
- moved D1 5.91 mm to (118.7, 111.1)
- moved C2 4.24 mm to (131.9, 104.9), turned to 90 degrees
- moved U2 4.00 mm to (126.0, 106.8)
- moved J3 3.98 mm to (109.0, 127.7)
- moved C1 3.41 mm to (122.8, 113.6)
- moved R1 2.30 mm to (135.4, 117.4), turned to 180 degrees
- moved J4 1.81 mm to (139.7, 113.5)
- moved C4 1.40 mm to (126.0, 129.4)
- moved U4 1.26 mm to (131.8, 141.5)
- moved C6 1.20 mm to (136.0, 141.2)
- moved J5 0.72 mm to (127.3, 145.4)
- turned D2 to -90 degrees
Connections:
- net Net-(C1-Pad1) renamed VIN
- U1 pad 20: unconnected-(U1-Pad20) -> PB7
- U1 pad 21: unconnected-(U1-Pad21) -> PD4
- U1 pad 22: unconnected-(U1-Pad22) -> PD5
- U1 pad 23: unconnected-(U1-Pad23) -> PD6
Routing:
- net PD6: track 0.00 -> 22.1 mm
- net VIN: track 10.3 -> 32.2 mm
- net PD5: track 0.00 -> 20.4 mm
- net PD4: track 0.00 -> 18.6 mm
- net PB7: track 0.00 -> 16.9 mm
- net LIGHT: track 8.30 -> 21.4 mm
- net +3V3: track 24.2 -> 29.8 mm, vias 8 -> 11
- net GND: track 19.5 -> 24.3 mm, vias 6 -> 9
- net SWIM: track 17.5 -> 21.8 mm
- net NRESET: track 36.9 -> 40.8 mm
- net Net-(J5-Pad1): track 10.2 -> 7.74 mm
- net Net-(J5-Pad2): track 6.94 -> 4.89 mm
- net I2C_SCL: track 10.7 -> 12.7 mm
- net SERIAL_INCOMING: track 13.7 -> 11.9 mm
- net Net-(J5-Pad3): track 5.21 -> 3.49 mm
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Other:
- board text added: "*"
- board text added: "+"
- board text added: "3.3"
- board text added: "4.6 to 12 volts"
- board text added: "GND"
- board text added: "LIGHT"
- board text added: "PB7"
- board text added: "PD4"
- board text added: "PD5"
- board text added: "PD6"
- board text added: "RX"
- board text added: "SERIAL"
- board text added: "SWIM"
- board text added: "TX"
- board text added: "VIN"
- board text added: "a2bikelight rev 1"
- board text added: "power"
