File: board/a2bikelight/a2bikelight.kicad_pcb (KiCad board)
At the start: 4 copper layers, 50 x 50 mm, 28 parts, among them J1 Barrel_Jack_Switch, J2 Conn_01x02_Male, J3 Conn_01x04_Male, J4 Conn_01x06_Male, J5 Conn_01x05_Male, J6 Conn_01x08_Male, SW1 SW_Push, SW2 SW_Push, U1 STM8L151K4U, U2 AMS1117-3.3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

Commit message: fet
Parts:
- added Q1: Si2301CDS, Package_TO_SOT_SMD:SOT-23, F.Cu at (161.6, 124.4)
- added Q1: Si2301CDS, Package_TO_SOT_SMD:SOT-23, F.Cu at (118.8, 122.6)
- added R3: 10k, Resistor_SMD:R_0805_2012Metric, F.Cu at (152.7, 128.5)
- added R4: 10, Resistor_SMD:R_2512_6332Metric, F.Cu at (154.8, 124.6)
- renumbered C6 to C5, C5 to C6, J5 to J7, R3 to R5, SW2 to SW1, SW1 to SW2

Commit message: rev2
Parts:
- removed C5: 100nF, Capacitor_SMD:C_0603_1608Metric
- removed J7: Conn_01x05_Male, Connector_PinHeader_2.54mm:PinHeader_1x05_P2.54mm_Vertical
- removed the Q1 at (118.8, 122.6)
- removed U4: MXC6655XA, Package_LGA:LGA-12_2x2mm_P0.5mm
- added J5: Conn_01x02_Male, Connector_PinHeader_2.54mm:PinHeader_1x02_P2.54mm_Vertical, F.Cu at (140.6, 132.9)
- moved SW1 21.3 mm to (131.7, 145.8), turned to 180 degrees
- moved R4 21.0 mm to (136.1, 134.2), turned to 90 degrees
- moved Q1 17.6 mm to (146.3, 133.1), turned to 90 degrees
- moved R3 10.4 mm to (146.1, 136.6), turned to 180 degrees
- moved D2 9.81 mm to (129.2, 136.3), turned to 90 degrees
- moved R5 5.92 mm to (129.2, 132.5)
Connections:
- U1 pad 11: unconnected-(U1-Pad11) -> LIGHT
- U1 pad 12: LIGHT -> unconnected-(U1-Pad12)
- U1 pad 33: thermal -> GND
Routing:
- net VIN: track 32.2 -> 60.2 mm
- net LIGHT: track 21.4 -> 46.1 mm
- net Net-(C5-Pad2): track 9.37 -> 0.00 mm
- net GND: track 24.3 -> 32.3 mm, vias 9 -> 17
- net Net-(J7-Pad1): track 7.74 -> 0.00 mm
- net Net-(C5-Pad1): track 7.69 -> 0.00 mm
- net Net-(J5-Pad1): track 0.00 -> 6.02 mm
- net BUTTON: track 25.2 -> 19.6 mm
- net Net-(J5-Pad2): track 0.00 -> 5.20 mm
- net Net-(J7-Pad2): track 4.89 -> 0.00 mm
- net Net-(J7-Pad3): track 3.49 -> 0.00 mm
- net Net-(D2-Pad2): track 3.64 -> 2.04 mm
- net PD4: track 18.6 -> 19.5 mm
Other:
- board text added: "PD3"
- board text added: "a2bikelight rev 2"
- board text added: "reset"
- board text added: "user button"
- board text removed: "PD4"
- board text removed: "a2bikelight rev 1"
